File: hardware/faout.sch (EAGLE design)
At the start: 169 parts, among them IC2 MT48LC8M16A2, Q1 12MHz, Q2 MUN2214T1, Q3 MUN2214T1, Q4 ASFL, SW1 SMD_TACT_SWITCH, SW2 SMD_TACT_SWITCH, SW3 SMD_TACT_SWITCH, U1 93LC46BT-I/OT, U10 REF102AU, U11 DAC8811DGK, U12 REF102AU, U13 DAC8811DGK, U14 ADR435ARZ, U15 AD8627AKSZ-R2, U16 OPA2277UA/2K5E4, U17 OPA2277UA/2K5E4, U18 MCP1700T-2502E/TT, U19 AD7980ARMZ, U2 LM3480IM3-3.3, U3 L7812ACV, U4 L7912ACV, U5 LM3671MF-3.3, U6 LM3671MF-1.2, U7 M25PE16, U8 6SLX9TQG144, U9 AD8220ARMZ

Commit message: WIP: Design 6channel FAOUT prototype.
Parts:
- removed AI1: BU-SMA, analog_out_lib:BU-SMA
- removed APWR: (no value), pinhead:PINHD-1X3
- removed C86, C87: 1uF, faout:C_EU0603
- removed DISP: 7SEG_DISPLAY, faout:7SEG_DISPLAY
- removed JTAG, P1: (no value), pinhead:PINHD-1X6
- removed LED1, LED2, LED3, LED4, LED5, PWR: (no value), led:LEDSML0805
- removed Q2, Q3: MUN2214T1, transistor-npn:MUN2214T1
- removed R29, R30: 2k, faout:R_EU0603
- removed RST: (no value), pinhead:PINHD-1X2
- removed SW1, SW2, SW3: SMD_TACT_SWITCH, faout:SMD_TACT_SWITCH
- removed U18: MCP1700T-2502E/TT, faout:MCP1700T-2502E/TT
- removed U19: AD7980ARMZ, faout:AD7980ARMZ
- added AO3, AO4, AO5, AO6: BU-SMA, analog_out_lib:BU-SMA
- C11: value 10uF -> 20pF; device faout:C_EU0805 -> faout:C_EU0603; OC_FARNELL 1867958 -> (none)
- C38: value 100uF -> 20pF; device rcl:CPOL-EUE -> faout:C_EU0603; OC_FARNELL 9693467 -> (none)
- C65, C66, C70, C73: value 100nF -> 1uF; OC_FARNELL 1740621 -> 1759409
- C68, C76, C77: value 100nF -> 20pF; OC_FARNELL 1740621 -> (none)
- C71: value 114pF -> 100nF; OC_FARNELL (none) -> 1740621
- C72: value 11.4pF -> 100nF; OC_FARNELL (none) -> 1740621
- C74: value 20pF -> 1uF; OC_FARNELL (none) -> 1759409
- C78, C79: value 1nF -> 1uF; OC_FARNELL (none) -> 1759409
- C85: value 22uF -> 1uF; device faout:C_EU1206 -> faout:C_EU0603; OC_FARNELL 1833823 -> 1759409
- R11, R15, R17: value 100 -> 5k
- R12, R13, R14, R16: value 100 -> 10k
- R21, R23: value 300 -> 5k
- R22, R24, R25, R7: value 300 -> 10k
- R26: value 7.47k -> 13.181k
- R27: value 7.47k -> 5k
- R28: value 134k -> 10k
- R8: value 0 -> 5k
- R9: value 0 -> 10k
- U11, U13: value DAC8811DGK -> OPA4277UA; device faout:DAC8811DGK -> faout:OPA4277UA
- U12: value REF102AU -> DAC8812; device faout:REF102AU -> faout:DAC8812
- U14: value ADR435ARZ -> REF102AU; device faout:ADR435ARZ -> faout:REF102AU
- U15: value AD8627AKSZ-R2 -> DAC8812; device faout:AD8627AKSZ-R2 -> faout:DAC8812
- U16: value OPA2277UA/2K5E4 -> OPA4277UA; device faout:OPA2277UA/2K5E4 -> faout:OPA4277UA
- U2: value LM3480IM3-3.3 -> REF102AU; device faout:LM3480IM3-3.3 -> faout:REF102AU
- U7: value M25PE16 -> M25PE16SO8N; device faout:M25PE16 -> faout:M25PE16SO8N
- U9: value AD8220ARMZ -> DAC8812; device faout:AD8220ARMZ -> faout:DAC8812
Connections:
- removed net 2V5: C84.P$1, U18.VOUT, U19.VDD
- removed net ADC1_CNV: U19.CNV, U8B1.IO_L33P_1
- removed net ADC1_REF: C85.P$1, U14.VOUT, U19.REF
- removed net ADC1_SCK: U19.SCK, U8B1.IO_L34P_1
- removed net ADC1_SDI: U19.SDI, U8B1.IO_L34N_1
- removed net ADC1_SDO: U19.SDO, U8B1.IO_L33N_1
- removed net BUTTON1: SW1.1, U8B2.IO_L12N_D2_MISO3_2
- removed net BUTTON2: SW2.1, U8B2.IO_L12P_D1_MISO2_2
- removed net BUTTON3: SW3.1, U8B2.IO_L2N_CMPMOSI_2
- removed net DAC1_IOUT: C74.P$2, U11.IOUT, U17.-IN_A
- removed net DAC1_VOUT: AO1.1, C74.P$1, U11.RFB, U17.OUT_A
- removed net DAC1_VREFOUT: C78.P$1, R29.P$2, U17.-IN_B
- removed net DAC2_IOUT: C75.P$2, U13.IOUT, U16.-IN_A
- removed net DAC2_VOUT: AO2.1, C75.P$1, U13.RFB, U16.OUT_A
- removed net DAC2_VREFOUT: C79.P$1, R30.P$2, U16.-IN_B
- removed net DISP_A: R14.P$2, U8B2.IO_L31N_GCLK30_D15_2
- removed net DISP_B: R13.P$2, U8B2.IO_L48P_D7_2
- removed net DISP_C: R12.P$2, U8B2.IO_L30P_GCLK1_D13_2
- removed net DISP_CAT1: DISP.CAT1@1, DISP.CAT1@2, Q3.C
- removed net DISP_CAT2: DISP.CAT2@1, DISP.CAT2@2, Q2.C
- removed net DISP_D: R11.P$2, U8B2.IO_L30N_GCLK0_USERCCLK_2
- removed net DISP_E: R17.P$2, U8B2.IO_L14N_D12_2
- removed net DISP_EN1: Q3.B, U8B2.IO_L14P_D11_2
- removed net DISP_EN2: Q2.B, U8B2.IO_L13N_D10_2
- removed net DISP_F: R16.P$2, U8B2.IO_L31P_GCLK31_D14_2
- removed net DISP_G: R15.P$2, U8B2.IO_L48N_RDWR_B_VREF_2
- removed net DISP_INT_A: DISP.A1, DISP.A2, R14.P$1
- removed net DISP_INT_B: DISP.B1, DISP.B2, R13.P$1
- removed net DISP_INT_C: DISP.C1, DISP.C2, R12.P$1
- removed net DISP_INT_D: DISP.D1, DISP.D2, R11.P$1
- removed net DISP_INT_E: DISP.E1, DISP.E2, R17.P$1
- removed net DISP_INT_F: DISP.F1, DISP.F2, R16.P$1
- removed net DISP_INT_G: DISP.G1, DISP.G2, R15.P$1
- removed net JP_1: P1.1, U8B1.IO_L43N_GCLK4_1
- removed net JP_2: P1.2, U8B1.IO_L45P_1
- removed net JP_3: P1.3, U8B1.IO_L45N_1
- removed net JP_4: P1.4, U8B1.IO_L46P_1
- removed net LED1: LED1.A, U8B1.IO_L46N_1
- removed net LED2: LED2.A, U8B1.IO_L47P_1
- removed net LED3: LED3.A, U8B1.IO_L47N_1
- removed net LED_4: LED4.A, U8B0.IO_L66P_SCP1_0
- removed net LED_5: LED5.A, U8B0.IO_L66N_SCP0_0
- removed net N$15: C72.P$1, R28.P$2, U15.+IN
- removed net N$17: C87.P$1, U10.NR
- removed net N$18: R18.P$1, SW1.2
- removed net N$19: R19.P$1, SW2.2
- removed net N$22: LED2.C, R22.P$2
- removed net N$23: LED3.C, R23.P$2
- removed net N$26: PWR.C, R7.P$2
- removed net N$27: C88.P$1, U12.NR
- removed net N$3: LED4.C, R24.P$2
- new net !DAC1_LDAC: U8B2.IO_L48P_D7_2, U9.~LDAC
- new net !DAC2_LDAC: U12.~LDAC, U8B2.IO_L30P_GCLK1_D13_2
- new net !DAC3_CS: U15.~CS, U8B1.IO_L43N_GCLK4_1
- new net !DAC3_LDAC: U15.~LDAC, U8B1.IO_L45P_1
- new net !DACX_RS: R28.P$1, U12.~RS, U15.~RS, U8B2.IO_L2P_CMPCLK_2, U9.~RS
- new net AGND: AO1.2, AO2.2, AO3.2, AO4.2, AO5.2, AO6.2, C1.P$2, C12.P$2, C13.P$1, C14.P$2, C15.P$1, C2.P$2, C6.P$2, C65.P$2, C66.P$2, C67.P$1, C69.P$2, C7.P$1, C70.P$2, C71.P$2, C72.P$1, C73.P$2, C74.P$1, C78.P$2, C79.P$2, C80.P$2, C81.P$1, C82.P$2, C83.P$1, C84.P$2, C85.P$1, C88.P$2, C89.+, C90.-, R27.P$2, R28.P$2, U10.COM, U11.+IN_A, U11.+IN_B, U11.+IN_C, U11.+IN_D, U12.AGNDA, U12.AGNDB, U12.DGND, U13.+IN_A, U13.+IN_B, U13.+IN_C, U13.+IN_D, U14.COM, U15.AGNDA, U15.AGNDB, U15.DGND, U16.+IN_A, U16.+IN_B, U16.+IN_C, U16.+IN_D, U17.V-, U2.COM, U3.GND, U4.GND, U9.AGNDA, U9.AGNDB, U9.DGND
- new net DAC1_IOUTA: C38.P$2, U11.-IN_B, U9.IOUTA
- new net DAC1_IOUTB: C75.P$2, U11.-IN_A, U9.IOUTB
- new net DAC1_RFBA: C38.P$1, R11.P$1, U11.OUT_B, U9.RFBA
- new net DAC1_RFBB: C75.P$1, R8.P$1, U11.OUT_A, U9.RFBB
- new net DAC1_VOUTA: AO1.1, R13.P$1, U11.OUT_C
- new net DAC1_VOUTB: AO2.1, R9.P$1, U11.OUT_D
- new net DAC2_IOUTA: C68.P$2, U12.IOUTA, U13.-IN_B
- new net DAC2_IOUTB: C11.P$2, U12.IOUTB, U13.-IN_A
- new net DAC2_RFBA: C68.P$1, R17.P$1, U12.RFBA, U13.OUT_B
- new net DAC2_RFBB: C11.P$1, R15.P$1, U12.RFBB, U13.OUT_A
- new net DAC2_VOUTA: AO3.1, R19.P$1, U13.OUT_C
- new net DAC2_VOUTB: AO4.1, R16.P$1, U13.OUT_D
- new net DAC3_CLK: U15.CLK, U8B1.IO_L45N_1
- new net DAC3_IOUTA: C77.P$2, U15.IOUTA, U16.-IN_B
- new net DAC3_IOUTB: C76.P$2, U15.IOUTB, U16.-IN_A
- new net DAC3_RFBA: C77.P$1, R23.P$1, U15.RFBA, U16.OUT_B
- new net DAC3_RFBB: C76.P$1, R21.P$1, U15.RFBB, U16.OUT_A
- new net DAC3_SDI: U15.SDI, U8B1.IO_L43P_GCLK5_1
- new net DAC3_VOUTA: AO5.1, R25.P$1, U16.OUT_C
- new net DAC3_VOUTB: AO6.1, R22.P$1, U16.OUT_D
- new net DAC3_VREF: R20.P$2, R24.P$2, U14.VOUT, U15.VREFA, U15.VREFB
- new net GPIO_0_0: U8B0.IO_L34P_GCLK19_0
- new net GPIO_0_1: U8B0.IO_L34N_GCLK18_0
- new net GPIO_0_2: U8B0.IO_L35P_GCLK17_0
- new net GPIO_0_3: U8B0.IO_L35N_GCLK16_0
- net !DAC1_CS: now also U8B2.IO_L31N_GCLK30_D15_2, U9.~CS; no longer U11.!CS, U8B1.IO_L40N_GCLK10_1
- net !DAC2_CS: now also U12.~CS, U8B2.IO_L14N_D12_2; no longer U13.!CS, U8B1.IO_L42P_GCLK7_1
- net !USB_OE: now also U8B0.IO_L66N_SCP0_0; no longer U8B0.IO_L64N_SCP4_0
- net !USB_RD: now also U8B0.IO_L65N_SCP2_0; no longer U8B0.IO_L63P_SCP7_0
- net !USB_RXF: now also U8B0.IO_L64N_SCP4_0; no longer U8B0.IO_L62P_0
- net !USB_TXE: now also U8B0.IO_L65P_SCP3_0; no longer U8B0.IO_L62N_VREF_0
- net !USB_WR: now also U8B0.IO_L66P_SCP1_0; no longer U8B0.IO_L63N_SCP6_0
- net +15V: no longer APWR.1, U2.IN
- net -15V: no longer APWR.2
- net 3V3: no longer C38.+, JTAG.6, P1.6, PWR.A, R18.P$2, R19.P$2, R20.P$2
- net 5V0: no longer R8.P$1
- net A+12V: now also C66.P$1, C69.P$1, C71.P$1, C78.P$1, C84.P$1, C88.P$1, R26.P$1, U10.V+, U11.V+, U13.V+, U14.V+, U2.V+; no longer C65.P$1, C76.P$1, U14.VIN, U15.V+, U9.+VS
- net A+3V3: now also U12.MSB, U12.VDD, U15.MSB, U15.VDD, U17.-IN_A, U17.OUT_A, U9.MSB, U9.VDD; no longer C11.P$1, C67.P$1, C68.P$1, C69.P$1, C70.P$1, C86.P$1, U10.V+, U11.VDD, U12.V+, U13.VDD, U18.VIN, U19.VIO, U2.OUT
- net A-12V: now also C67.P$2, C72.P$2, C74.P$2, C85.P$2, U11.V-, U13.V-; no longer C66.P$2, C77.P$2, U15.V-, U17.V-, U9.-VS
- net DAC1_CLK: now also U8B2.IO_L48N_RDWR_B_VREF_2, U9.CLK; no longer U11.CLK, U8B1.IO_L41P_GCLK9_IRDY1_1
- net DAC1_SDI: now also U8B2.IO_L31P_GCLK31_D14_2, U9.SDI; no longer U11.SDI, U8B1.IO_L41N_GCLK8_1
- net DAC1_VREF: now also R12.P$2, R7.P$2, U10.VOUT, U9.VREFA, U9.VREFB; no longer C78.P$2, U10.COM, U11.VREF, U17.OUT_B
- net DAC2_CLK: now also U12.CLK, U8B2.IO_L30N_GCLK0_USERCCLK_2; no longer U13.CLK, U8B1.IO_L42N_GCLK6_TRDY1_1
- net DAC2_SDI: now also U12.SDI, U8B2.IO_L14P_D11_2; no longer U13.SDI, U8B1.IO_L43P_GCLK5_1
- net DAC2_VREF: now also R14.P$2, R18.P$2, U12.VREFA, U12.VREFB, U2.VOUT; no longer C79.P$2, U12.COM, U13.VREF, U16.OUT_B
- net GND: no longer AO1.2, AO2.2, APWR.3, C1.P$2, C11.P$2, C12.P$2, C13.P$1, C14.P$2, C15.P$1, C2.P$2, C38.-, C6.P$2, C65.P$2, C66.P$1, C67.P$2, C68.P$2, C69.P$2, C7.P$1, C70.P$2, C72.P$2, C73.P$2, C76.P$2, C77.P$1, C80.P$2, C81.P$1, C82.P$2, C83.P$1, C84.P$2, C85.P$2, C86.P$2, C87.P$2, C88.P$2, C89.+, C90.-, JTAG.1, P1.5, Q2.E, Q3.E, R21.P$1, R22.P$1, R23.P$1, R24.P$1, R25.P$1, R27.P$1, R7.P$1, R9.P$1, RST.2, SW1.3, SW1.4, SW2.3, SW2.4, SW3.3, SW3.4, U11.GND, U13.GND, U14.GND, U16.+IN_A, U16.+IN_B, U17.+IN_A, U17.+IN_B, U18.GND, U19.GND, U19.IN-, U2.GND, U3.GND, U4.GND, U9.REF
- net N$10: now also R20.P$1, R21.P$2, R22.P$2, U16.-IN_D; no longer R29.P$1, U10.VOUT
- net N$11: now also C70.P$1, U2.NR; no longer AI1.2, U9.-IN
- net N$12: now also C79.P$1, U14.NR; no longer C71.P$1, U15.-IN, U15.OUT_A, U19.IN+
- net N$13: now also R27.P$1, U17.+IN_A; no longer U9.VOUT
- net N$14: now also R23.P$2, R24.P$1, R25.P$2, U16.-IN_C; no longer C71.P$2, R26.P$1, R27.P$2, R28.P$1
- net N$20: now also R17.P$2, R18.P$1, R19.P$2, U13.-IN_C; no longer R20.P$1, SW3.2
- net N$21: now also R14.P$1, R15.P$2, R16.P$2, U13.-IN_D; no longer LED1.C, R21.P$2
- net N$4: now also C65.P$1, U10.NR; no longer LED5.C, R25.P$2
- net N$8: now also R11.P$2, R12.P$1, R13.P$2, U11.-IN_C; no longer R30.P$1, U12.VOUT
- net N$9: now also R7.P$1, R8.P$2, R9.P$2, U11.-IN_D; no longer AI1.1, U9.+IN
- net RAM_A8: now also U8B2.IO_L64N_D9_2; no longer U8B2.IO_L64P_D8_2
- net RAM_A9: now also U8B2.IO_L64P_D8_2; no longer U8B2.IO_L64N_D9_2
- net RESET: no longer RST.1
- net TCK: no longer JTAG.2
- net TDI: no longer JTAG.3
- net TDO: no longer JTAG.4
- net TMS: no longer JTAG.5
- net USB_D0: now also U8B0.IO_L36P_GCLK15_0; no longer U8B0.IO_L64P_SCP5_0
- net USB_D1: now also U8B0.IO_L36N_GCLK14_0; no longer U8B0.IO_L34P_GCLK19_0
- net USB_D2: now also U8B0.IO_L37P_GCLK13_0; no longer U8B0.IO_L34N_GCLK18_0
- net USB_D3: now also U8B0.IO_L62P_0; no longer U8B0.IO_L35P_GCLK17_0
- net USB_D4: now also U8B0.IO_L62N_VREF_0; no longer U8B0.IO_L35N_GCLK16_0
- net USB_D5: now also U8B0.IO_L63P_SCP7_0; no longer U8B0.IO_L36P_GCLK15_0
- net USB_D6: now also U8B0.IO_L63N_SCP6_0; no longer U8B0.IO_L36N_GCLK14_0
- net USB_D7: now also U8B0.IO_L64P_SCP5_0; no longer U8B0.IO_L37P_GCLK13_0
- net USB_GND: no longer R9.P$2
- net USB_V: no longer R8.P$2
Other:
- note removed: "1MHz Filter"
- note removed: "Analog in"
- note removed: "FPGA User IO"
- moved on the sheet: AO1, AO2, C11, C40, C41, C42, C43, C44, C45, C46, C47, C48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

Commit message: WIP: Compress FAOUT-6 layout to 7cm, use space for connectors.
Parts:
- removed L3: (no value), faout:R_EU0603
- removed L4, L5: 2.2uH, rcl:L-EUL5038P
- removed U16: OPA4277UA, faout:OPA4277UA
- removed U17: OPA2277UA/2K5E4, faout:OPA2277UA/2K5E4
- removed USB_RST: (no value), pinhead:PINHD-1X2
- added C86: 1uF, faout:C_EU0603
- added C87, C91: 100nF, faout:C_EU0603
- added P1: TE_CONN_MTE_HEADER3R, faout:TE_CONN_MTE_HEADER3R
- added Q2: L7912ACV, faout:L7912ACV
- added Q3: 12MHz, faout:TXC_QUARTZ_7A
- added R29, R30, R31, R34, R35: 10k, faout:R_EU0603
- added R32, R33: 5k, faout:R_EU0603
- added SV1: (no value), con-ml:ML6L
- added SV2: (no value), con-ml:ML10
- C1, C12, C13, C2: value 10uF -> 4.7uF; device faout:C_EU0805 -> faout:C_EU0603; OC_FARNELL 1867958 -> 1833803
- C11: value 20pF -> 4.7uF; OC_FARNELL (none) -> 1833803
- C14: value 10uF -> 100nF; device faout:C_EU0805 -> faout:C_EU0603; OC_FARNELL 1867958 -> 1740621
- C16, C7: value 100nF -> 10uF; device faout:C_EU0603 -> faout:C_EU0805; OC_FARNELL 1740621 -> 1867958
- C17, C9: value 100nF -> 100uF; device faout:C_EU0603 -> rcl:CPOL-EUE; OC_FARNELL 1740621 -> 9693467
- C18, C8: value 4.7uF -> 10uF; device faout:C_EU0603 -> faout:C_EU0805; OC_FARNELL 1833803 -> 1867958
- C20: value 100nF -> 4.7uF; OC_FARNELL 1740621 -> 1833803
- C21, C22: value 4.7uF -> 100nF; OC_FARNELL 1833803 -> 1740621
- C29, C30: value 470nF -> 100nF; OC_FARNELL 1867949 -> 1740621
- C3: value 3.3uF -> 4.7uF
- C31: value 4.7uF -> 3.3uF
- C32, C33: value 4.7uF -> 18pF; OC_FARNELL 1833803 -> (none)
- C34, C35, C43, C44, C46, C49, C56: value 4.7uF -> 470nF; OC_FARNELL 1833803 -> 1867949
- C37, C59: value 10nF -> 4.7uF; OC_FARNELL 1759102 -> 1833803
- C38: value 20pF -> 10nF; OC_FARNELL (none) -> 1759102
- C4: value 18pF -> 4.7uF; OC_FARNELL (none) -> 1833803
- C42, C48, C54, C60, C62: value 470nF -> 4.7uF; OC_FARNELL 1867949 -> 1833803
- C5: value 18pF -> 10uF; device faout:C_EU0603 -> faout:C_EU0805; OC_FARNELL (none) -> 1867958
- C64: value 4.7uF -> 10nF; OC_FARNELL 1833803 -> 1759102
- C68, C75, C76, C77: value 20pF -> 1uF; OC_FARNELL (none) -> 1759409
- C69, C70, C73, C78, C79, C88: value 1uF -> 100nF; OC_FARNELL 1759409 -> 1740621
- C71, C72, C80, C81: value 100nF -> 20pF; OC_FARNELL 1740621 -> (none)
- C83: value 100nF -> 1uF; OC_FARNELL 1740621 -> 1759409
- C89, C90: value 100uF -> 20pF; device rcl:CPOL-EUE -> faout:C_EU0603; OC_FARNELL 9693467 -> (none)
- L1, L2: value (none) -> 2.2uH; device faout:R_EU0603 -> rcl:L-EUL5038P; OC_FARNELL (none) -> 2145272
- Q1: value 12MHz -> L7812ACV; device faout:TXC_QUARTZ_7A -> faout:L7812ACV; OC_FARNELL 1841940 -> (none)
- R1, R2: value 10k -> ferrite; device faout:R_EU0603 -> faout:R_EU1206
- R10: value 4.7k -> 10k
- R11, R15, R23: value 5k -> 10k
- R13: value 10k -> 2.2k
- R14: value 10k -> 4.7k
- R16: value 10k -> 13.181k
- R20: value 10k -> 5k
- R26: value 13.181k -> 5k
- R3: value 2.2k -> ferrite; device faout:R_EU0603 -> faout:R_EU1206
- R4, R5: value 10k -> ferrite
- R6: value 12k -> 10k
- R7: value 10k -> NC
- R8: value 5k -> 12k
- R9: value 10k -> (none)
- U1: value 93LC46BT-I/OT -> LM3671MF-3.3; device faout:93LC46BT-I/OT -> faout:LM3671MF-3.3
- U13: value OPA4277UA -> REF102AU; device faout:OPA4277UA -> faout:REF102AU
- U14: value REF102AU -> OPA4277UA; device faout:REF102AU -> faout:OPA4277UA
- U2: value REF102AU -> LM3671MF-1.2; device faout:REF102AU -> faout:LM3671MF-1.2
- U3: value L7812ACV -> 93LC46BT-I/OT; device faout:L7812ACV -> faout:93LC46BT-I/OT
- U4: value L7912ACV -> 6SLX9TQG144; device faout:L7912ACV -> faout:6SLX9TQG144; OC_FARNELL (none) -> 1876228
- U5: value LM3671MF-3.3 -> M25PE16SO8N; device faout:LM3671MF-3.3 -> faout:M25PE16SO8N
- U6: value LM3671MF-1.2 -> OPA2277UA/2K5E4; device faout:LM3671MF-1.2 -> faout:OPA2277UA/2K5E4
- U7: value M25PE16SO8N -> REF102AU; device faout:M25PE16SO8N -> faout:REF102AU
- U8: value 6SLX9TQG144 -> OPA4277UA; device faout:6SLX9TQG144 -> faout:OPA4277UA; OC_FARNELL 1876228 -> (none)
Connections:
- removed net N$16: L1.P$1, USB1.SHD@4
- new net N$15: R9.P$1, USB1.SHD@4
- new net P1_1: SV2.1, U4B1.IO_L42P_GCLK7_1
- new net P1_2: SV2.2, U4B1.IO_L42N_GCLK6_TRDY1_1
- new net P1_3: SV2.3, U4B1.IO_L41P_GCLK9_IRDY1_1
- new net P1_4: SV2.4, U4B1.IO_L41N_GCLK8_1
- new net P1_5: SV2.5, U4B1.IO_L33P_1
- new net P1_6: SV2.6, U4B1.IO_L33N_1
- new net P1_7: SV2.7, U4B1.IO_L32P_1
- new net P1_8: SV2.8, U4B1.IO_L32N_1
- net !DAC1_CS: now also U4B2.IO_L31N_GCLK30_D15_2; no longer U8B2.IO_L31N_GCLK30_D15_2
- net !DAC1_LDAC: now also U4B2.IO_L48P_D7_2; no longer U8B2.IO_L48P_D7_2
- net !DAC2_CS: now also U4B2.IO_L14N_D12_2; no longer U8B2.IO_L14N_D12_2
- net !DAC2_LDAC: now also U4B2.IO_L30P_GCLK1_D13_2; no longer U8B2.IO_L30P_GCLK1_D13_2
- net !DAC3_CS: now also U4B1.IO_L46N_1; no longer U8B1.IO_L43N_GCLK4_1
- net !DAC3_LDAC: now also U4B1.IO_L47P_1; no longer U8B1.IO_L45P_1
- net !DACX_RS: now also R15.P$1, U4B2.IO_L2P_CMPCLK_2; no longer R28.P$1, U8B2.IO_L2P_CMPCLK_2
- net !RAM_CAS: now also U4B3.IO_L52N_3; no longer U8B3.IO_L52N_3
- net !RAM_RAS: now also U4B3.IO_L83P_3; no longer U8B3.IO_L83P_3
- net !RAM_WE: now also U4B3.IO_L52P_3; no longer U8B3.IO_L52P_3
- net !USB_OE: now also U4B0.IO_L66N_SCP0_0; no longer U8B0.IO_L66N_SCP0_0
- net !USB_RD: now also U4B0.IO_L65N_SCP2_0; no longer U8B0.IO_L65N_SCP2_0
- net !USB_RESET: now also R6.P$1, R7.P$1; no longer R5.P$1, USB_RST.1
- net !USB_RXF: now also U4B0.IO_L64N_SCP4_0; no longer U8B0.IO_L64N_SCP4_0
- net !USB_TXE: now also U4B0.IO_L65P_SCP3_0; no longer U8B0.IO_L65P_SCP3_0
- net !USB_WR: now also U4B0.IO_L66P_SCP1_0; no longer U8B0.IO_L66P_SCP1_0
- net +15V: now also C5.P$1, P1.1, Q1.IN; no longer C1.P$1, U3.IN
- net -15V: now also C18.P$1, P1.2, Q2.IN; no longer C2.P$1, U4.IN
- net 1V2: now also C12.P$1, C13.P$1, C52.P$1, C53.P$1, C54.P$1, C55.P$1, L2.2, U2.FB, U4BVCCINT.VCCINT@0, U4BVCCINT.VCCINT@1, U4BVCCINT.VCCINT@2, U4BVCCINT.VCCINT@3, U4BVCCINT.VCCINT@4; no longer C33.P$1, C36.P$1, C41.P$1, C43.P$1, C45.P$1, C46.P$1, L5.2, U6.FB, U8BVCCINT.VCCINT@0, U8BVCCINT.VCCINT@1, U8BVCCINT.VCCINT@2, U8BVCCINT.VCCINT@3, U8BVCCINT.VCCINT@4
- net 1V8: now also C25.P$1, C31.P$1; no longer C20.P$1, C3.P$1
- net 3V3: now also C3.P$1, C36.P$1, C38.P$1, C4.P$1, C41.P$1, C43.P$1, C45.P$1, C46.P$1, L1.2, R11.P$2, R12.P$2, R14.P$2, R4.P$1, R5.P$1, R6.P$2, SV2.10, U1.FB, U2.EN, U3.VCC, U4B0.VCCO_0@0, U4B0.VCCO_0@1, U4B0.VCCO_0@2, U4B1.VCCO_1@0, U4B1.VCCO_1@1, U4B1.VCCO_1@2, U4B2.IO_L1N_M0_CMPMISO_2, U4B2.VCCO_2@0, U4B2.VCCO_2@1, U4B3.VCCO_3@0, U4B3.VCCO_3@1, U4B3.VCCO_3@2, U4BVCCAUX.VCCAUX@0, U4BVCCAUX.VCCAUX@1, U4BVCCAUX.VCCAUX@2, U4BVCCAUX.VCCAUX@3, U4BVCCAUX.VCCAUX@4, U5.!RESET, U5.!WP, U5.VCC; no longer C25.P$1, C31.P$1, C32.P$1, C52.P$1, C53.P$1, C54.P$1, C55.P$1, C9.P$1, L2.P$1, L3.P$1, L4.2, R1.P$2, R2.P$2, R4.P$2, R5.P$2, U1.VCC, U5.FB, U6.EN, U7.!RESET, U7.!WP, U7.VCC, U8B0.VCCO_0@0, U8B0.VCCO_0@1, U8B0.VCCO_0@2, U8B1.VCCO_1@0, U8B1.VCCO_1@1, U8B1.VCCO_1@2, U8B2.IO_L1N_M0_CMPMISO_2, U8B2.VCCO_2@0, U8B2.VCCO_2@1, U8B3.VCCO_3@0, U8B3.VCCO_3@1, U8B3.VCCO_3@2, U8BVCCAUX.VCCAUX@0, U8BVCCAUX.VCCAUX@1, U8BVCCAUX.VCCAUX@2, U8BVCCAUX.VCCAUX@3, U8BVCCAUX.VCCAUX@4
- net 5V0: now also C1.P$1, C10.P$1, C11.P$1, C2.P$1, R1.P$2, U1.EN, U1.VIN, U2.VIN; no longer C18.P$1, C19.P$1, C21.P$1, C22.P$1, U5.EN, U5.VIN, U6.VIN
- net A+12V: now also C65.P$1, C67.P$1, C7.P$1, C74.P$1, C76.P$1, C8.P$1, C83.P$1, C85.P$1, C87.P$1, C9.+, Q1.OUT, R16.P$1, U6.V+, U7.V+, U8.V+; no longer C12.P$1, C14.P$1, C66.P$1, C71.P$1, C73.P$1, C80.P$1, C82.P$1, C84.P$1, C88.P$1, C90.+, R26.P$1, U16.V+, U17.V+, U2.V+, U3.OUT
- net A+3V3: now also C73.P$1, C82.P$1, C91.P$1, U6.-IN_A, U6.OUT_A; no longer U17.-IN_A, U17.OUT_A
- net A-12V: now also C14.P$2, C16.P$2, C17.-, C68.P$2, C70.P$2, C77.P$2, C79.P$2, C86.P$2, C88.P$2, Q2.OUTPUT, U14.V-, U8.V-; no longer C13.P$2, C67.P$2, C7.P$2, C72.P$2, C74.P$2, C81.P$2, C83.P$2, C85.P$2, C89.-, U13.V-, U16.V-, U4.OUTPUT
- net AGND: now also C14.P$1, C16.P$1, C17.+, C18.P$2, C5.P$2, C67.P$2, C68.P$1, C7.P$2, C70.P$1, C74.P$2, C75.P$2, C76.P$2, C77.P$1, C79.P$1, C8.P$2, C83.P$2, C85.P$2, C86.P$1, C87.P$2, C88.P$1, C9.-, C91.P$2, P1.3, Q1.GND, Q2.GND, R15.P$2, R17.P$2, R2.P$1, U13.COM, U14.+IN_A, U14.+IN_B, U14.+IN_C, U14.+IN_D, U6.V-, U7.COM, U8.+IN_A, U8.+IN_B, U8.+IN_C, U8.+IN_D; no longer C1.P$2, C12.P$2, C13.P$1, C14.P$2, C2.P$2, C67.P$1, C7.P$1, C70.P$2, C71.P$2, C72.P$1, C74.P$1, C79.P$2, C80.P$2, C81.P$1, C83.P$1, C85.P$1, C88.P$2, C89.+, C90.-, R27.P$2, R28.P$2, U13.+IN_A, U13.+IN_B, U13.+IN_C, U13.+IN_D, U14.COM, U16.+IN_A, U16.+IN_B, U16.+IN_C, U16.+IN_D, U17.V-, U2.COM, U3.GND, U4.GND
- net CLK_IN: now also U4B1.IO_L40P_GCLK11_1; no longer U8B1.IO_L40P_GCLK11_1
- net DAC1_CLK: now also U4B2.IO_L48N_RDWR_B_VREF_2; no longer U8B2.IO_L48N_RDWR_B_VREF_2
- net DAC1_IOUTA: now also C72.P$2, U8.-IN_B; no longer C38.P$2, U11.-IN_B
- net DAC1_IOUTB: now also C71.P$2, U8.-IN_A; no longer C75.P$2, U11.-IN_A
- net DAC1_RFBA: now also C72.P$1, R21.P$1, U8.OUT_B; no longer C38.P$1, R11.P$1, U11.OUT_B
- net DAC1_RFBB: now also C71.P$1, R20.P$1, U8.OUT_A; no longer C75.P$1, R8.P$1, U11.OUT_A
- net DAC1_SDI: now also U4B2.IO_L31P_GCLK31_D14_2; no longer U8B2.IO_L31P_GCLK31_D14_2
- net DAC1_VOUTA: now also R23.P$1, U8.OUT_C; no longer R13.P$1, U11.OUT_C
- net DAC1_VOUTB: now also R19.P$1, U8.OUT_D; no longer R9.P$1, U11.OUT_D
- net DAC1_VREF: now also R18.P$2, R22.P$2, U7.VOUT; no longer R12.P$2, R7.P$2, U10.VOUT
- net DAC2_CLK: now also U4B2.IO_L30N_GCLK0_USERCCLK_2; no longer U8B2.IO_L30N_GCLK0_USERCCLK_2
- net DAC2_IOUTA: now also C81.P$2, U11.-IN_B; no longer C68.P$2, U13.-IN_B
- net DAC2_IOUTB: now also C80.P$2, U11.-IN_A; no longer C11.P$2, U13.-IN_A
- net DAC2_RFBA: now also C81.P$1, R27.P$1, U11.OUT_B; no longer C68.P$1, R17.P$1, U13.OUT_B
- net DAC2_RFBB: now also C80.P$1, R26.P$1, U11.OUT_A; no longer C11.P$1, R15.P$1, U13.OUT_A
- net DAC2_SDI: now also U4B2.IO_L14P_D11_2; no longer U8B2.IO_L14P_D11_2
- net DAC2_VOUTA: now also R29.P$1, U11.OUT_C; no longer R19.P$1, U13.OUT_C
- net DAC2_VOUTB: now also R25.P$1, U11.OUT_D; no longer R16.P$1, U13.OUT_D
- net DAC2_VREF: now also R24.P$2, R28.P$2, U10.VOUT; no longer R14.P$2, R18.P$2, U2.VOUT
- net DAC3_CLK: now also U4B1.IO_L47N_1; no longer U8B1.IO_L45N_1
- net DAC3_IOUTA: now also C90.P$2, U14.-IN_B; no longer C77.P$2, U16.-IN_B
- net DAC3_IOUTB: now also C89.P$2, U14.-IN_A; no longer C76.P$2, U16.-IN_A
- net DAC3_RFBA: now also C90.P$1, R33.P$1, U14.OUT_B; no longer C77.P$1, R23.P$1, U16.OUT_B
- net DAC3_RFBB: now also C89.P$1, R32.P$1, U14.OUT_A; no longer C76.P$1, R21.P$1, U16.OUT_A
- net DAC3_SDI: now also U4B1.IO_L46P_1; no longer U8B1.IO_L43P_GCLK5_1
- net DAC3_VOUTA: now also R35.P$1, U14.OUT_C; no longer R25.P$1, U16.OUT_C
- net DAC3_VOUTB: now also R31.P$1, U14.OUT_D; no longer R22.P$1, U16.OUT_D
- net DAC3_VREF: now also R30.P$2, R34.P$2, U13.VOUT; no longer R20.P$2, R24.P$2, U14.VOUT
- net EECS: now also R10.P$1, U3.CS; no longer R1.P$1, U1.CS
- net EEDATA: now also R12.P$1, R13.P$1, U3.DI; no longer R3.P$1, R4.P$1, U1.DI
- net EESK: now also R11.P$1, U3.CLK; no longer R2.P$1, U1.CLK
- net FLASH_CS: now also U4B2.IO_L65N_CSO_B_2, U5.!CS; no longer U7.!CS, U8B2.IO_L65N_CSO_B_2
- net FLASH_MISO: now also U4B2.IO_L3P_D0_DIN_MISO_MISO1_2, U5.SDO; no longer U7.SDO, U8B2.IO_L3P_D0_DIN_MISO_MISO1_2
- net FLASH_MOSI: now also U4B2.IO_L3N_MOSI_CSI_B_MISO0_2, U5.SDI; no longer U7.SDI, U8B2.IO_L3N_MOSI_CSI_B_MISO0_2
- net FLASH_SCK: now also U4B2.IO_L1P_CCLK_2, U5.SCK; no longer U7.SCK, U8B2.IO_L1P_CCLK_2
- net GND: now also C1.P$2, C11.P$2, C12.P$2, C13.P$2, C2.P$2, C38.P$2, R2.P$2, R3.P$2, R7.P$2, R8.P$2, SV1.5, SV1.6, SV2.9, U2.GND, U3.GND, U4B0.IO_L1P_HSWAPEN_0, U4B1.IO_L1N_VREF_1, U4B1.IO_L1P_1, U4B1.IO_L34N_1, U4B1.IO_L34P_1, U4B1.IO_L40N_GCLK10_1, U4B1.IO_L43N_GCLK4_1, U4B1.IO_L43P_GCLK5_1, U4B1.IO_L45N_1, U4B1.IO_L45P_1, U4B2.IO_L12N_D2_MISO3_2, U4B2.IO_L12P_D1_MISO2_2, U4B2.IO_L13N_D10_2, U4B2.IO_L13P_M1_2, U4B2.IO_L2N_CMPMOSI_2, U4B3.IO_L1N_VREF_3, U4BGND.GND@0, U4BGND.GND@1, U4BGND.GND@10, U4BGND.GND@11, U4BGND.GND@12, U4BGND.GND@2, U4BGND.GND@3, U4BGND.GND@4, U4BGND.GND@5, U4BGND.GND@6, U4BGND.GND@7, U4BGND.GND@8, U4BGND.GND@9, U4BNA.SUSPEND; no longer C16.P$2, C17.P$2, C18.P$2, C5.P$2, C8.P$2, C9.P$2, L1.P$2, R6.P$2, U6.GND, U7.GND, U8B0.IO_L1P_HSWAPEN_0, U8B2.IO_L13P_M1_2, U8BGND.GND@0, U8BGND.GND@1, U8BGND.GND@10, U8BGND.GND@11, U8BGND.GND@12, U8BGND.GND@2, U8BGND.GND@3, U8BGND.GND@4, U8BGND.GND@5, U8BGND.GND@6, U8BGND.GND@7, U8BGND.GND@8, U8BGND.GND@9, U8BNA.SUSPEND, USB_RST.2
- net GPIO_0_0: now also SV1.1, U4B0.IO_L34P_GCLK19_0; no longer U8B0.IO_L34P_GCLK19_0
- net GPIO_0_1: now also SV1.2, U4B0.IO_L34N_GCLK18_0; no longer U8B0.IO_L34N_GCLK18_0
- net GPIO_0_2: now also SV1.3, U4B0.IO_L35P_GCLK17_0; no longer U8B0.IO_L35P_GCLK17_0
- net GPIO_0_3: now also SV1.4, U4B0.IO_L35N_GCLK16_0; no longer U8B0.IO_L35N_GCLK16_0
- net N$1: now also C32.P$1, Q3.P$1; no longer C4.P$1, Q1.P$1
- net N$10: now also R30.P$1, R31.P$2, R32.P$2, U14.-IN_D; no longer R20.P$1, R21.P$2, R22.P$2, U16.-IN_D
- net N$11: now also C75.P$1, U10.NR; no longer C70.P$1, U2.NR
- net N$12: now also C84.P$1, U13.NR; no longer C79.P$1, U14.NR
- net N$13: now also R16.P$2, R17.P$1, U6.+IN_A; no longer R26.P$2, R27.P$1, U17.+IN_A
- net N$14: now also R33.P$2, R34.P$1, R35.P$2, U14.-IN_C; no longer R23.P$2, R24.P$1, R25.P$2, U16.-IN_C
- net N$2: now also C33.P$1, Q3.P$2; no longer C5.P$1, Q1.P$2
- net N$20: now also R27.P$2, R28.P$1, R29.P$2, U11.-IN_C; no longer R17.P$2, R18.P$1, R19.P$2, U13.-IN_C
- net N$21: now also R24.P$1, R25.P$2, R26.P$2, U11.-IN_D; no longer R14.P$1, R15.P$2, R16.P$2, U13.-IN_D
- net N$24: now also L1.1, U1.SW; no longer L4.1, U5.SW
- net N$25: now also L2.1, U2.SW; no longer L5.1, U6.SW
- net N$4: now also C66.P$1, U7.NR; no longer C65.P$1, U10.NR
- net N$5: now also C19.P$1, C21.P$1, R5.P$2; no longer C16.P$1, C8.P$1, L3.P$2
- net N$6: now also R13.P$2, U3.DO; no longer R3.P$2, U1.DO
- net N$7: now also C20.P$1, C22.P$1, R4.P$2; no longer C10.P$1, C17.P$1, L2.P$2
- net N$8: now also R21.P$2, R22.P$1, R23.P$2, U8.-IN_C; no longer R11.P$2, R12.P$1, R13.P$2, U11.-IN_C
- net N$9: now also R18.P$1, R19.P$2, R20.P$2, U8.-IN_D; no longer R7.P$1, R8.P$2, R9.P$2, U11.-IN_D
- net RAM_A0: now also U4B0.IO_L3P_0; no longer U8B0.IO_L3P_0
- net RAM_A1: now also U4B0.IO_L3N_0; no longer U8B0.IO_L3N_0
- net RAM_A10: now also U4B0.IO_L2N_0; no longer U8B0.IO_L2N_0
- net RAM_A11: now also U4B3.IO_L1P_3; no longer U8B3.IO_L1P_3
- net RAM_A2: now also U4B0.IO_L4P_0; no longer U8B0.IO_L4P_0
- net RAM_A3: now also U4B0.IO_L4N_0; no longer U8B0.IO_L4N_0
- net RAM_A4: now also U4B2.IO_L49P_D3_2; no longer U8B2.IO_L49P_D3_2
- net RAM_A5: now also U4B2.IO_L49N_D4_2; no longer U8B2.IO_L49N_D4_2
- net RAM_A6: now also U4B2.IO_L62P_D5_2; no longer U8B2.IO_L62P_D5_2
- net RAM_A7: now also U4B2.IO_L62N_D6_2; no longer U8B2.IO_L62N_D6_2
- net RAM_A8: now also U4B2.IO_L64N_D9_2; no longer U8B2.IO_L64N_D9_2
- net RAM_A9: now also U4B2.IO_L64P_D8_2; no longer U8B2.IO_L64P_D8_2
- net RAM_BA0: now also U4B0.IO_L1N_VREF_0; no longer U8B0.IO_L1N_VREF_0
- net RAM_BA1: now also U4B0.IO_L2P_0; no longer U8B0.IO_L2P_0
- net RAM_CKE: now also U4B3.IO_L2P_3; no longer U8B3.IO_L2P_3
- net RAM_CLK: now also U4B3.IO_L2N_3; no longer U8B3.IO_L2N_3
- net RAM_CS: now also U4B3.IO_L83N_VREF_3; no longer U8B3.IO_L83N_VREF_3
- net RAM_DQ0: now also U4B3.IO_L50N_3; no longer U8B3.IO_L50N_3
- net RAM_DQ1: now also U4B3.IO_L50P_3; no longer U8B3.IO_L50P_3
- net RAM_DQ10: now also U4B3.IO_L41N_GCLK26_3; no longer U8B3.IO_L41N_GCLK26_3
- net RAM_DQ11: now also U4B3.IO_L41P_GCLK27_3; no longer U8B3.IO_L41P_GCLK27_3
- net RAM_DQ12: now also U4B3.IO_L37N_3; no longer U8B3.IO_L37N_3
- net RAM_DQ13: now also U4B3.IO_L37P_3; no longer U8B3.IO_L37P_3
- net RAM_DQ14: now also U4B3.IO_L36N_3; no longer U8B3.IO_L36N_3
- net RAM_DQ15: now also U4B3.IO_L36P_3; no longer U8B3.IO_L36P_3
- net RAM_DQ2: now also U4B3.IO_L49N_3; no longer U8B3.IO_L49N_3
- net RAM_DQ3: now also U4B3.IO_L49P_3; no longer U8B3.IO_L49P_3
- net RAM_DQ4: now also U4B3.IO_L44N_GCLK20_3; no longer U8B3.IO_L44N_GCLK20_3
- net RAM_DQ5: now also U4B3.IO_L44P_GCLK21_3; no longer U8B3.IO_L44P_GCLK21_3
- net RAM_DQ6: now also U4B3.IO_L43N_GCLK22_IRDY2_3; no longer U8B3.IO_L43N_GCLK22_IRDY2_3
- net RAM_DQ7: now also U4B3.IO_L51P_3; no longer U8B3.IO_L51P_3
- net RAM_DQ8: now also U4B3.IO_L42N_GCLK24_3; no longer U8B3.IO_L42N_GCLK24_3
- net RAM_DQ9: now also U4B3.IO_L42P_GCLK25_TRDY2_3; no longer U8B3.IO_L42P_GCLK25_TRDY2_3
- net RAM_DQMH: now also U4B3.IO_L43P_GCLK23_3; no longer U8B3.IO_L43P_GCLK23_3
- net RAM_DQML: now also U4B3.IO_L51N_3; no longer U8B3.IO_L51N_3
- net RESET: now also R14.P$1, U4B2.PROGRAM_B_2; no longer R10.P$1, U8B2.PROGRAM_B_2
- net TCK: now also U4BNA.TCK; no longer U8BNA.TCK
- net TDI: now also U4BNA.TDI; no longer U8BNA.TDI
- net TDO: now also U4BNA.TDO; no longer U8BNA.TDO
- net TMS: now also U4BNA.TMS; no longer U8BNA.TMS
- net USB_CLKOUT: now also U4B0.IO_L37N_GCLK12_0; no longer U8B0.IO_L37N_GCLK12_0
- net USB_D0: now also U4B0.IO_L36P_GCLK15_0; no longer U8B0.IO_L36P_GCLK15_0
- net USB_D1: now also U4B0.IO_L36N_GCLK14_0; no longer U8B0.IO_L36N_GCLK14_0
- net USB_D2: now also U4B0.IO_L37P_GCLK13_0; no longer U8B0.IO_L37P_GCLK13_0
- net USB_D3: now also U4B0.IO_L62P_0; no longer U8B0.IO_L62P_0
- net USB_D4: now also U4B0.IO_L62N_VREF_0; no longer U8B0.IO_L62N_VREF_0
- net USB_D5: now also U4B0.IO_L63P_SCP7_0; no longer U8B0.IO_L63P_SCP7_0
- net USB_D6: now also U4B0.IO_L63N_SCP6_0; no longer U8B0.IO_L63N_SCP6_0
- net USB_D7: now also U4B0.IO_L64P_SCP5_0; no longer U8B0.IO_L64P_SCP5_0
- net USB_GND: now also R3.P$1, R9.P$2
- net USB_REF: now also R8.P$1; no longer R6.P$1
- net USB_V: now also R1.P$1
Other:
- note added: "Connectors"
- moved on the sheet: AO1, AO2, AO3, AO4, AO5, AO6, C1, C10, C11, C12, C13, C14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
